File: pcb/knobdeavour.kicad_pcb (KiCad board)
At the start: 2 copper layers, 224.4 x 97.8 mm, 102 parts, among them J0 USB_C_Receptacle_USB2.0, J1 BREAKOUT, J2 Conn_01x03_Male, J3 Conn_01x02_Female, J4 Conn_01x01_Male, K1 KEYSW, K10 KEYSW, K11 KEYSW, K12 KEYSW, K13 KEYSW, K14 KEYSW, K15 KEYSW, K16 KEYSW, K17 KEYSW, K18 KEYSW, K19 KEYSW, K2 KEYSW, K20 KEYSW, K24 KEYSW, K25 KEYSW, K26 KEYSW, K27 KEYSW, K28 KEYSW, K29 KEYSW, K3 KEYSW, K30 KEYSW, K31 KEYSW, K32 KEYSW, K33 KEYSW, K34 KEYSW, K35 KEYSW, K36 KEYSW, K37 KEYSW, K38 KEYSW, K39 KEYSW, K4 KEYSW, K40 KEYSW, K41 KEYSW, K5 KEYSW, K6 KEYSW, K7 KEYSW, K8 KEYSW, K9 KEYSW, SW1 RotaryEncoder_Switch, SW2 RotaryEncoder_Switch, SW3 SW_PUSH, SW4 RESET, U1 NCP1117-3.3_SOT223, U2 W25Q128JVS, U3 RP2040, U44 SRV05-4, Y0 12MHZ Crystal

Commit message: rows routed
Parts:
- moved C17 2.51 mm to (162.9, 56.7)
- moved C4 2.51 mm to (162.9, 54.5)
Routing:
- net Net-(D21-Pad1): track 100.7 -> 139.3 mm
- net Net-(D9-Pad1): track 14.7 -> 36.3 mm
- net Net-(D5-Pad2): track 37.7 -> 57.0 mm
- net Net-(D5-Pad1): track 61.4 -> 79.5 mm
- net Net-(D1-Pad2): track 83.4 -> 100.7 mm
- net Net-(D2-Pad2): track 101.4 -> 115.4 mm
- net Net-(D16-Pad2): track 28.3 -> 14.7 mm
- net GND: track 322.6 -> 309.0 mm, vias 16 -> 15
- net Net-(D2-Pad1): track 84.1 -> 97.2 mm
- net Net-(D6-Pad2): track 67.8 -> 80.0 mm
- net Net-(D8-Pad1): track 33.3 -> 21.4 mm
- net Net-(D7-Pad1): track 61.4 -> 72.8 mm
- net Net-(D6-Pad1): track 50.0 -> 61.0 mm
- net Net-(D1-Pad1): track 130.8 -> 122.6 mm
- net +3V3: track 183.6 -> 178.0 mm, vias 4 -> 3
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